Commit message: Fixed depth

File: drivers/jaco2_driver/urdf/j2n6s300.urdf.xacro (robot description, xacro)
@@ -15,5 +15,5 @@
 	xmlns:xacro="http://www.ros.org/wiki/xacro" name="j2n6s300">
   <xacro:include filename="$(find kinova_description)/urdf/j2n6s300.xacro"/>
-    <xacro:property name="M_PI" value="3.14159"/>
+  <xacro:property name="M_PI" value="3.14159"/>
   <link name="root"/>
   <!-- for gazebo -->
@@ -21,4 +21,11 @@
   <link name="left_arm_mount"/>
   <link name="right_arm_mount"/>
+  <link name="kinect">
+    <visual>
+      <geometry>
+        <mesh filename="package://jaco2_driver/meshes/kinect.dae"/>
+      </geometry>
+    </visual>
+  </link>
   <joint name="connect_root_and_world" type="fixed">
     <child link="root" />
@@ -29,13 +36,17 @@
     <child link="left_arm_mount" />
     <parent link="root" />
-    <origin xyz="0.0261046 0.13335 0.2799937" rpy="${-M_PI/2} 0 ${-M_PI/2}"/>
+    <origin xyz="-0.15675 0.13335 0.0" rpy="${-M_PI/2} 0 ${-M_PI/2}"/>
   </joint>
   <joint name="right_arm_attach" type="fixed">
     <child link="right_arm_mount" />
     <parent link="root" />
-    <origin xyz="0.0261046 -0.13335 0.2799937" rpy="${-M_PI/2} 0 ${-M_PI/2}" />
+    <origin xyz="-0.15675 -0.13335 0.0" rpy="${-M_PI/2} 0 ${-M_PI/2}" />
+  </joint>
+  <joint name="kinect_attach" type="fixed">
+    <child link="kinect" />
+    <parent link="root" />
+    <origin xyz="0.125 0.0 0.3" rpy="0.0 0.0 0.0" />
   </joint>
   <xacro:property name="robot_root" value="root" />
-n
   <xacro:j2n6s300 base_parent="left_arm_mount" prefix="left"/>
   <xacro:j2n6s300 base_parent="right_arm_mount" prefix="right"/>
